Commit message: Add Isaac Sim back-end: SICK S300 lasers, self-collision fix, nav docs
- isaac_sim/: mir_isaac_sim.py bridge (PhysX + RTX SICK S300 lidars), USD
  assets, conversion scripts, README_isaac.md
- mir_isaac.launch.py (RSP + ros2_control + MoveIt + RViz + scan merger) and
  mir_isaac_scan_merger.launch.py
- diffdrive_controller_isaac.yaml with enable_odom_tf=false (Isaac bridge
  publishes odom->base via --publish-odom); Gazebo's diffdrive_controller.yaml
  restored to enable_odom_tf=true so its nav works
- lidar self-collision unblock so the merged /scan covers full 360 like Gazebo
- README: Isaac Sim demo section, portability/paths notes, screenshot

Co-Authored-By: Claude Opus 4.8 <noreply@anthropic.com>
Claude-Session: https://claude.ai/code/session_01NQzvPQRQXzHfe6K69R8hry

File: Universal_Robots_ROS2_Description/urdf/ur.ros2_control.xacro (robot description, xacro)
@@ -6,4 +6,7 @@
     sim_gazebo:=false
     sim_ignition:=false
+    sim_isaac:=false
+    isaac_joint_commands:=/isaac_joint_commands
+    isaac_joint_states:=/isaac_joint_states
     headless_mode:=false
     initial_positions:=${dict(shoulder_pan_joint=0.0,shoulder_lift_joint=-1.57,elbow_joint=0.0,wrist_1_joint=-1.57,wrist_2_joint=0.0,wrist_3_joint=0.0)}
@@ -30,4 +33,10 @@
           <plugin>ign_ros2_control/IgnitionSystem</plugin>
         </xacro:if>
+        <xacro:if value="${sim_isaac}">
+          <plugin>topic_based_ros2_control/TopicBasedSystem</plugin>
+          <param name="joint_commands_topic">${isaac_joint_commands}</param>
+          <param name="joint_states_topic">${isaac_joint_states}</param>
+          <param name="sum_wrapped_joint_states">true</param>
+        </xacro:if>
         <xacro:if value="${use_fake_hardware}">
           <plugin>mock_components/GenericSystem</plugin>
@@ -36,5 +45,5 @@
           <param name="calculate_dynamics">true</param>
         </xacro:if>
-        <xacro:unless value="${use_fake_hardware or sim_gazebo or sim_ignition}">
+        <xacro:unless value="${use_fake_hardware or sim_gazebo or sim_ignition or sim_isaac}">
           <plugin>ur_robot_driver/URPositionHardwareInterface</plugin>
           <param name="robot_ip">${robot_ip}</param>
@@ -125,5 +134,5 @@
         <state_interface name="effort"/>
       </joint>
-      <xacro:unless value="${sim_gazebo or sim_ignition}">
+      <xacro:unless value="${sim_gazebo or sim_ignition or sim_isaac}">
         <sensor name="${tf_prefix}tcp_fts_sensor">
           <state_interface name="force.x"/>

File: Universal_Robots_ROS2_Description/urdf/ur_macro.xacro (robot description, xacro)
@@ -62,4 +62,7 @@
     sim_gazebo:=false
     sim_ignition:=false
+    sim_isaac:=false
+    isaac_joint_commands:=/isaac_joint_commands
+    isaac_joint_states:=/isaac_joint_states
     headless_mode:=false
     initial_positions:=${dict(shoulder_pan_joint=0.0,shoulder_lift_joint=-1.57,elbow_joint=0.0,wrist_1_joint=-1.57,wrist_2_joint=0.0,wrist_3_joint=0.0)}
@@ -104,4 +107,7 @@
         sim_gazebo="${sim_gazebo}"
         sim_ignition="${sim_ignition}"
+        sim_isaac="${sim_isaac}"
+        isaac_joint_commands="${isaac_joint_commands}"
+        isaac_joint_states="${isaac_joint_states}"
         script_filename="${script_filename}"
         output_recipe_filename="${output_recipe_filename}"

File: mir_robot/mir_description/urdf/include/mir_100_v1.urdf.xacro (robot description, xacro)
@@ -200,4 +200,7 @@
     <xacro:arg name="sim_gazebo" default="true" />
     <xacro:arg name="sim_ignition" default="false" />
+    <xacro:arg name="sim_isaac" default="false" />
+    <xacro:arg name="isaac_joint_commands" default="/isaac_joint_commands" />
+    <xacro:arg name="isaac_joint_states" default="/isaac_joint_states" />
     <xacro:arg name="simulation_controllers" default="" />
     <!-- initial position for simulations (Fake Hardware, Gazebo, Ignition) -->
@@ -229,4 +232,7 @@
       sim_gazebo="$(arg sim_gazebo)"
       sim_ignition="$(arg sim_ignition)"
+      sim_isaac="$(arg sim_isaac)"
+      isaac_joint_commands="/isaac_arm_commands"
+      isaac_joint_states="$(arg isaac_joint_states)"
       headless_mode="$(arg headless_mode)"
       initial_positions="${xacro.load_yaml(initial_positions_file)}"
@@ -328,5 +334,5 @@
   <!-- Import gripper macros -->
   <xacro:include filename="$(find mir_description)/urdf/include/robotiq_gripper_macro.xacro" />
-  <xacro:robotiq_gripper name="RobotiqGripperHardwareInterface" prefix="" parent="ur_tool0" use_fake_hardware="$(arg use_fake_hardware)" com_port="$(arg com_port)" sim_gazebo="$(arg sim_gazebo)">
+  <xacro:robotiq_gripper name="RobotiqGripperHardwareInterface" prefix="" parent="ur_tool0" use_fake_hardware="$(arg use_fake_hardware)" com_port="$(arg com_port)" sim_gazebo="$(arg sim_gazebo)" sim_isaac="$(arg sim_isaac)" isaac_joint_commands="/isaac_gripper_commands" isaac_joint_states="$(arg isaac_joint_states)">
     <origin xyz="0 0 0" rpy="0 0 0" />
   </xacro:robotiq_gripper>

File: mir_robot/mir_description/urdf/include/robotiq_gripper.ros2_control.xacro (robot description, xacro)
@@ -58,10 +58,26 @@
                 <state_interface name="velocity"/>
             </joint>
-            <!-- When simulating we need to include the rest of the gripper joints -->
-            <xacro:if value="${sim_gazebo or use_fake_hardware or sim_isaac or sim_ignition}">
+            <!-- When simulating we need to include the rest of the gripper joints.
+                 NOTE: sim_isaac is deliberately EXCLUDED here. Under Isaac these
+                 mimic joints would be listed with NO command/state interface (see
+                 the inner <xacro:unless> below). topic_based_ros2_control 0.2.0
+                 mishandles such interface-less mimic joints and corrupts the heap
+                 in TopicBasedSystem (ros2_control_node aborts with
+                 "free(): invalid next size"), so no joint state is ever read.
+                 For Isaac we therefore emit ONLY the master knuckle joint above;
+                 PhysX couples the mimic joints and robot_state_publisher still
+                 visualizes them via the URDF <mimic> tags from the master joint. -->
+            <xacro:if value="${sim_gazebo or use_fake_hardware or sim_ignition}">
                 <joint name="${prefix}robotiq_85_right_knuckle_joint">
                     <param name="mimic">${prefix}robotiq_85_left_knuckle_joint</param>
                     <param name="multiplier">-1</param>
-                    <xacro:unless value="${sim_ignition}">
+                    <!-- Isaac couples the mimic joints in PhysX (like Ignition),
+                         so it must NOT also command them: a command interface here
+                         makes TopicBasedSystem publish all 6 joints, and the
+                         bridge's ArticulationController then fights the PhysX mimic
+                         (fingers splay). Exclude command/state for sim_isaac too;
+                         robot_state_publisher still visualizes them via the URDF
+                         <mimic> tags from the master joint. -->
+                    <xacro:unless value="${sim_ignition or sim_isaac}">
                         <command_interface name="position"/>
                         <state_interface name="position"/>
@@ -72,5 +88,12 @@
                     <param name="mimic">${prefix}robotiq_85_left_knuckle_joint</param>
                     <param name="multiplier">1</param>
-                    <xacro:unless value="${sim_ignition}">
+                    <!-- Isaac couples the mimic joints in PhysX (like Ignition),
+                         so it must NOT also command them: a command interface here
+                         makes TopicBasedSystem publish all 6 joints, and the
+                         bridge's ArticulationController then fights the PhysX mimic
+                         (fingers splay). Exclude command/state for sim_isaac too;
+                         robot_state_publisher still visualizes them via the URDF
+                         <mimic> tags from the master joint. -->
+                    <xacro:unless value="${sim_ignition or sim_isaac}">
                         <command_interface name="position"/>
                         <state_interface name="position"/>
@@ -81,5 +104,12 @@
                     <param name="mimic">${prefix}robotiq_85_left_knuckle_joint</param>
                     <param name="multiplier">-1</param>
-                    <xacro:unless value="${sim_ignition}">
+                    <!-- Isaac couples the mimic joints in PhysX (like Ignition),
+                         so it must NOT also command them: a command interface here
+                         makes TopicBasedSystem publish all 6 joints, and the
+                         bridge's ArticulationController then fights the PhysX mimic
+                         (fingers splay). Exclude command/state for sim_isaac too;
+                         robot_state_publisher still visualizes them via the URDF
+                         <mimic> tags from the master joint. -->
+                    <xacro:unless value="${sim_ignition or sim_isaac}">
                         <command_interface name="position"/>
                         <state_interface name="position"/>
@@ -90,5 +120,12 @@
                     <param name="mimic">${prefix}robotiq_85_left_knuckle_joint</param>
                     <param name="multiplier">-1</param>
-                    <xacro:unless value="${sim_ignition}">
+                    <!-- Isaac couples the mimic joints in PhysX (like Ignition),
+                         so it must NOT also command them: a command interface here
+                         makes TopicBasedSystem publish all 6 joints, and the
+                         bridge's ArticulationController then fights the PhysX mimic
+                         (fingers splay). Exclude command/state for sim_isaac too;
+                         robot_state_publisher still visualizes them via the URDF
+                         <mimic> tags from the master joint. -->
+                    <xacro:unless value="${sim_ignition or sim_isaac}">
                         <command_interface name="position"/>
                         <state_interface name="position"/>
@@ -99,5 +136,12 @@
                     <param name="mimic">${prefix}robotiq_85_left_knuckle_joint</param>
                     <param name="multiplier">1</param>
-                    <xacro:unless value="${sim_ignition}">
+                    <!-- Isaac couples the mimic joints in PhysX (like Ignition),
+                         so it must NOT also command them: a command interface here
+                         makes TopicBasedSystem publish all 6 joints, and the
+                         bridge's ArticulationController then fights the PhysX mimic
+                         (fingers splay). Exclude command/state for sim_isaac too;
+                         robot_state_publisher still visualizes them via the URDF
+                         <mimic> tags from the master joint. -->
+                    <xacro:unless value="${sim_ignition or sim_isaac}">
                         <command_interface name="position"/>
                         <state_interface name="position"/>

File: mir_robot/mir_description/urdf/mir.urdf.xacro (robot description, xacro)
@@ -22,7 +22,15 @@
     left_wheel_joint="${prefix}left_wheel_joint"
     right_wheel_joint="${prefix}right_wheel_joint"/>  -->
-  <ros2_control name="GazeboSystem" type="system">
+  <ros2_control name="MiRBaseSystem" type="system">
     <hardware>
-      <plugin>gazebo_ros2_control/GazeboSystem</plugin>
+      <xacro:if value="$(arg sim_isaac)">
+        <plugin>topic_based_ros2_control/TopicBasedSystem</plugin>
+        <param name="joint_commands_topic">/isaac_base_commands</param>
+        <param name="joint_states_topic">$(arg isaac_joint_states)</param>
+        <param name="sum_wrapped_joint_states">true</param>
+      </xacro:if>
+      <xacro:unless value="$(arg sim_isaac)">
+        <plugin>gazebo_ros2_control/GazeboSystem</plugin>
+      </xacro:unless>
     </hardware>
     <joint name="left_wheel_joint">
@@ -42,42 +50,56 @@
       <state_interface name="velocity"/>
     </joint>
-    <joint name="fl_caster_rotation_joint">
-      <state_interface name="position"/>
-      <state_interface name="velocity"/>
-    </joint>
-    <joint name="fr_caster_rotation_joint">
-      <state_interface name="position"/>
-      <state_interface name="velocity"/>
-    </joint>
-    <joint name="bl_caster_rotation_joint">
-      <state_interface name="position"/>
-      <state_interface name="velocity"/>
-    </joint>
-    <joint name="br_caster_rotation_joint">
-      <state_interface name="position"/>
-      <state_interface name="velocity"/>
-    </joint>
-    <joint name="fl_caster_wheel_joint">
-      <state_interface name="position"/>
-      <state_interface name="velocity"/>
-    </joint>
-    <joint name="fr_caster_wheel_joint">
-      <state_interface name="position"/>
-      <state_interface name="velocity"/>
-    </joint>
-    <joint name="bl_caster_wheel_joint">
-      <state_interface name="position"/>
-      <state_interface name="velocity"/>
-    </joint>
-    <joint name="br_caster_wheel_joint">
-      <state_interface name="position"/>
-      <state_interface name="velocity"/>
-    </joint>
+    <!-- The passive casters are state-only joints. Under Isaac we must NOT list
+         them here: TopicBasedSystem then publishes /isaac_base_commands with
+         name=[10 joints] but velocity=[2 wheels] (a JointState whose name length
+         != value length), and Isaac's ROS2SubscribeJointState silently DROPS any
+         such inconsistent message -> the drive wheels never receive a command.
+         Dropping the casters from ros2_control makes the command message
+         name=2/velocity=2 (consistent), so it is delivered. The casters still
+         swivel/roll passively in Isaac; their joint state is just not fed back
+         through ros2_control (cosmetic, not used by nav/MoveIt). Gazebo keeps
+         them. -->
+    <xacro:unless value="$(arg sim_isaac)">
+      <joint name="fl_caster_rotation_joint">
+        <state_interface name="position"/>
+        <state_interface name="velocity"/>
+      </joint>
+      <joint name="fr_caster_rotation_joint">
+        <state_interface name="position"/>
+        <state_interface name="velocity"/>
+      </joint>
+      <joint name="bl_caster_rotation_joint">
+        <state_interface name="position"/>
+        <state_interface name="velocity"/>
+      </joint>
+      <joint name="br_caster_rotation_joint">
+        <state_interface name="position"/>
+        <state_interface name="velocity"/>
+      </joint>
+      <joint name="fl_caster_wheel_joint">
+        <state_interface name="position"/>
+        <state_interface name="velocity"/>
+      </joint>
+      <joint name="fr_caster_wheel_joint">
+        <state_interface name="position"/>
+        <state_interface name="velocity"/>
+      </joint>
+      <joint name="bl_caster_wheel_joint">
+        <state_interface name="position"/>
+        <state_interface name="velocity"/>
+      </joint>
+      <joint name="br_caster_wheel_joint">
+        <state_interface name="position"/>
+        <state_interface name="velocity"/>
+      </joint>
+    </xacro:unless>
   </ros2_control>
-  <gazebo>
-    <!-- Joint state publisher -->
-    <plugin filename="libgazebo_ros2_control.so" name="gazebo_ros2_control">
-      <parameters>$(find mir_description)/config/diffdrive_controller.yaml</parameters>
-    </plugin>
-  </gazebo>
+  <xacro:unless value="$(arg sim_isaac)">
+    <gazebo>
+      <!-- Joint state publisher -->
+      <plugin filename="libgazebo_ros2_control.so" name="gazebo_ros2_control">
+        <parameters>$(find mir_description)/config/diffdrive_controller.yaml</parameters>
+      </plugin>
+    </gazebo>
+  </xacro:unless>
 </robot>
