Commit message: Fix Gazebo base velocity tracking and switch local planner to MPPI
The simulated base never executed cmd_vel correctly: gazebo_ros2_control
applies a velocity command open loop, so the drive wheels ran a constant
+0.37 rad/s fast. The real MiR closes a velocity loop in its motor drives;
the sim had no equivalent. Adding vel_kp/vel_ki to the wheel joints fixes it.

Measured with Gazebo ground truth (/gazebo/link_states), before -> after:
  distance covered      115%  -> 102% of commanded
  straight-line drift   +7.0  -> -0.6..-2.6 deg over 1.8 m
  in-place rotation      23%  -> 104% of commanded
  creep at zero command 22.8  -> 0.6 mm/s
  spawn position error  metres -> 1.5 cm

Aligned the platform with the official MiR100 specification: 1.5 m/s
forwards, 0.3 m/s backwards, 24 rad/s at the wheel joints, and an
890 x 580 mm footprint (was 900 x 500, i.e. 80 mm too narrow).

Local planner switched from DWB to MPPI. DWB drives the whole lower half of
the maze correctly and then stalls at the 1.1 m gap, which needs a tighter
turn than the 1.3 m MiR100 requires for a U-turn; reducing inflation_radius
does not help, so inflation stays at the stock 0.6. MPPI completes the
traverse repeatedly and tracks 3-4x tighter on open paths (cross-track RMS:
straight 0.24 vs 1.08 cm, corner 1.35 vs 3.56 cm, circle 0.66 vs 2.23 cm),
at the cost of ~50% more time and noticeably more CPU. The DWB block is
kept commented out; swapping the two blocks reverts it.

PathAlignCritic.use_path_orientations must stay false while the global
planner is NavFn, which leaves intermediate pose orientations at identity.

Also fixed, all of which independently blocked navigation in simulation:
  - robot_x/y/yaw were declared but never reached spawn_entity
  - robot_description was not wrapped in ParameterValue(value_type=str), so
    any ':' in a URDF comment broke the launch
  - the UR5 and gripper had no controller: the arm collapsed into the front
    laser plane and Nav2 saw its own gripper as an obstacle inside the
    footprint, while the loose gripper fingers shook the base along at
    0.15 m/s
  - the merged /scan used the default range_max (inf), so nav2 never
    raytrace-cleared stale obstacles
  - velocity_smoother subscribed to its own output in navigation.py
  - librealsense_gazebo_plugin threw on load and randomly took gzserver
    with it; now off by default
  - maze.world had stray text after </sdf>

gazebo_debug.md records the diagnosis and, more usefully, the traps that
cost the most time: a stale robot_state_publisher silently serving an old
/robot_description, and XML comments inside <gazebo> or <ros2_control>
blocks segfaulting gzserver.

Co-Authored-By: Claude Opus 5 <noreply@anthropic.com>
Claude-Session: https://claude.ai/code/session_01CNPGJaYKhbsgFE1tUvVa9E

File: mir_robot/mir_description/urdf/include/common_properties.urdf.xacro (robot description, xacro)
@@ -84,3 +84,8 @@
     </inertial>
   </xacro:macro>
+  <!-- Torsional (spin about the contact normal) friction on the drive wheels.
+       Exposed as a property because it looks like it should govern how well the
+       base turns; measured with ground truth it does not. 300, 1.0 and 0.0 all
+       give an identical 23% of the commanded in-place rotation rate. -->
+  <xacro:property name="mir_wheel_torsional" value="300" />
 </robot>

File: mir_robot/mir_description/urdf/include/mir_100_v1.urdf.xacro (robot description, xacro)
@@ -204,6 +204,9 @@
     <xacro:arg name="isaac_joint_states" default="/isaac_joint_states" />
     <xacro:arg name="simulation_controllers" default="" />
-    <!-- initial position for simulations (Fake Hardware, Gazebo, Ignition) -->
-    <xacro:arg name="initial_positions_file" default="$(find ur_description)/config/initial_positions.yaml"/>
+    <!-- Initial position for simulations (Fake Hardware, Gazebo, Ignition).
+         Defaults to the stow pose rather than ur_description's arm-straight-out
+         pose, so the arm does not have to swing across the base right after
+         spawn. See mir_description/config/ur_stow_positions.yaml. -->
+    <xacro:arg name="initial_positions_file" default="$(find mir_description)/config/ur_stow_positions.yaml"/>
     <!-- convert to property to use substitution in function -->
     <xacro:property name="initial_positions_file" default="$(arg initial_positions_file)"/>
@@ -271,4 +274,10 @@
         </plugin>
       </gazebo>
+      <!-- gazebo_grasp_fix reports "Link ... can't be found in gazebo ...
+           Skipping" for several of the gripper links it is told to watch, so it
+           is only partly initialised. Set grasp_fix_plugin:=false to leave it
+           out (nothing else in the sim depends on it). -->
+      <xacro:arg name="grasp_fix_plugin" default="true" />
+      <xacro:if value="$(arg grasp_fix_plugin)">
       <gazebo>
         <plugin name="gazebo_grasp_fix" filename="libgazebo_grasp_fix.so">
@@ -295,4 +304,5 @@
         </plugin>
       </gazebo>
+      </xacro:if>
     </xacro:if>
     <xacro:if value="$(arg sim_ignition)">
@@ -327,5 +337,11 @@
       <origin xyz="0.035 0.05 0.03" rpy="0 ${pi} ${0.5 * pi}" />
     </joint>
-    <xacro:sensor_d435i parent="ur_flange" name="realsense" use_nominal_extrinsics="true">
+    <!-- realsense_gazebo_plugin is off by default: it throws during Load and
+         regularly segfaults gzserver right afterwards, while never actually
+         publishing colour or depth. Pass realsense_gazebo_plugin:=true if you
+         have a working build of it. -->
+    <xacro:arg name="realsense_gazebo_plugin" default="false" />
+    <xacro:sensor_d435i parent="ur_flange" name="realsense" use_nominal_extrinsics="true"
+                        add_gazebo_plugin="$(arg realsense_gazebo_plugin)">
       <origin xyz="0.02 0 -0.061" rpy="${pi} 0 0"/>
     </xacro:sensor_d435i>

File: mir_robot/mir_description/urdf/include/wheel.urdf.xacro (robot description, xacro)
@@ -8,5 +8,5 @@
       <child link="${prefix}${locationprefix}_wheel_link" />
       <axis xyz="0 1 0" />
-      <limit effort="100" velocity="20.0" />
+      <limit effort="100" velocity="24.0" />
       <!-- <dynamics damping="0.0" friction="0.0"/> -->
       <!-- <gazebo reference="${prefix}${locationprefix}_wheel_joint">
@@ -51,5 +51,5 @@
               </ode>
               <torsional>
-                <coefficient>300</coefficient>
+                <coefficient>${mir_wheel_torsional}</coefficient>
                 <use_patch_radius>false</use_patch_radius>
                 <surface_radius>${mir_100_act_wheel_radius}</surface_radius>

File: mir_robot/mir_description/urdf/mir.urdf.xacro (robot description, xacro)
@@ -34,19 +34,32 @@
       </xacro:unless>
     </hardware>
+    <!-- Wheel command limits are in rad/s at the joint, not m/s at the base.
+         0.8 m/s (the nav max_vel_x) needs 0.8 / 0.0625 = 12.8 rad/s, so the old
+         +-1 rad/s limit was an order of magnitude below what navigation asks
+         for. MiR100 tops out at 1.5 m/s = 24 rad/s, which is what the joint
+         limit and these bounds are set to. -->
     <joint name="left_wheel_joint">
       <command_interface name="velocity">
-        <param name="min">-1</param>
-        <param name="max">1</param>
+        <param name="min">-24</param>
+        <param name="max">24</param>
       </command_interface>
       <state_interface name="position"/>
       <state_interface name="velocity"/>
+      <param name="vel_kp">100.0</param>
+      <param name="vel_ki">20.0</param>
+      <param name="vel_kd">0.0</param>
+      <param name="vel_max_integral_error">10.0</param>
     </joint>
     <joint name="right_wheel_joint">
       <command_interface name="velocity">
-        <param name="min">-1</param>
-        <param name="max">1</param>
+        <param name="min">-24</param>
+        <param name="max">24</param>
       </command_interface>
       <state_interface name="position"/>
       <state_interface name="velocity"/>
+      <param name="vel_kp">100.0</param>
+      <param name="vel_ki">20.0</param>
+      <param name="vel_kd">0.0</param>
+      <param name="vel_max_integral_error">10.0</param>
     </joint>
     <!-- The passive casters are state-only joints. Under Isaac we must NOT list

File: realsense2_description/urdf/_d435i.urdf.xacro (robot description, xacro)
@@ -23,9 +23,16 @@
   <xacro:include filename="$(find realsense2_description)/urdf/_d435i_imu_modules.urdf.xacro"/>
   <xacro:include filename="$(find realsense2_description)/urdf/_d435i_gazebo.xacro"/>
-  <xacro:macro name="sensor_d435i" params="parent *origin name:=camera use_nominal_extrinsics:=false">
+  <!-- add_gazebo_plugin: set false to build the camera's links, frames and IMU
+       but leave out librealsense_gazebo_plugin. That plugin throws during Load
+       ("Exception occured in the Load function of plugin with name[camera]")
+       and frequently takes gzserver down with a segfault immediately after. It
+       publishes no colour or depth either way, so leaving it out only removes
+       the random crashes. -->
+  <xacro:macro name="sensor_d435i" params="parent *origin name:=camera use_nominal_extrinsics:=false add_gazebo_plugin:=true">
     <xacro:sensor_d435 parent="${parent}" name="${name}" use_nominal_extrinsics="${use_nominal_extrinsics}">
       <xacro:insert_block name="origin" />
     </xacro:sensor_d435>
     <xacro:d435i_imu_modules name="${name}" use_nominal_extrinsics="${use_nominal_extrinsics}"/>
+    <xacro:if value="${add_gazebo_plugin}">
     <xacro:gazebo_d435i camera_name="${name}"
                         topics_ns="camera"
@@ -54,4 +61,5 @@
                         visualize="true"
     />
+    </xacro:if>
   </xacro:macro>
 </robot>
