Commit message: Align Isaac navigation with Gazebo maze behavior

File: isaac_sim/mir_isaac.urdf (robot description, URDF)
Before this commit: robot mir_100, 58 links, 57 joints
Links:
- link back_laser_link: geometry collision mesh filename=/mnt/data/mir_isaac/install/mir_description/share/mir_descr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; visual mesh filename=/mnt/data/mir_isaac/install/mir_description/share/mir_descr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
- link base_link: geometry collision mesh filename=/mnt/data/mir_isaac/install/mir_description/share/mir_descr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; visual mesh filename=/mnt/data/mir_isaac/install/mir_description/share/mir_descr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
- link bl_caster_rotation_link: geometry collision mesh filename=/mnt/data/mir_isaac/install/mir_description/share/mir_descr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; visual mesh filename=/mnt/data/mir_isaac/install/mir_description/share/mir_descr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
- link bl_caster_wheel_link: geometry collision cylinder length=0.032 radius=0.0625; visual mesh filename=/mnt/data/mir_isaac/install/mir_description/share/mir_descr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
- link br_caster_rotation_link: geometry collision mesh filename=/mnt/data/mir_isaac/install/mir_description/share/mir_descr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; visual mesh filename=/mnt/data/mir_isaac/install/mir_description/share/mir_descr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
- link br_caster_wheel_link: geometry collision cylinder length=0.032 radius=0.0625; visual mesh filename=/mnt/data/mir_isaac/install/mir_description/share/mir_descr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
- link camera_mount: geometry collision mesh filename=/mnt/data/mir_isaac/install/mir_description/share/mir_descr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 scale=0.001 0.001 0.001; visual mesh filename=/mnt/data/mir_isaac/install/mir_description/share/mir_descr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 scale=0.001 0.001 0.001
- link fl_caster_rotation_link: geometry collision mesh filename=/mnt/data/mir_isaac/install/mir_description/share/mir_descr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; visual mesh filename=/mnt/data/mir_isaac/install/mir_description/share/mir_descr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
- link fl_caster_wheel_link: geometry collision cylinder length=0.032 radius=0.0625; visual mesh filename=/mnt/data/mir_isaac/install/mir_description/share/mir_descr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
- link fr_caster_rotation_link: geometry collision mesh filename=/mnt/data/mir_isaac/install/mir_description/share/mir_descr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; visual mesh filename=/mnt/data/mir_isaac/install/mir_description/share/mir_descr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
- link fr_caster_wheel_link: geometry collision cylinder length=0.032 radius=0.0625; visual mesh filename=/mnt/data/mir_isaac/install/mir_description/share/mir_descr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
- link front_laser_link: geometry collision mesh filename=/mnt/data/mir_isaac/install/mir_description/share/mir_descr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; visual mesh filename=/mnt/data/mir_isaac/install/mir_description/share/mir_descr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
- link left_wheel_link: geometry collision cylinder length=0.032 radius=0.0625; visual mesh filename=/mnt/data/mir_isaac/install/mir_description/share/mir_descr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
- link realsense_link: geometry collision box size=0.02505 0.09 0.025; visual mesh filename=/mnt/data/mir_isaac/install/realsense2_description/share/re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
- link right_wheel_link: geometry collision cylinder length=0.032 radius=0.0625; visual mesh filename=/mnt/data/mir_isaac/install/mir_description/share/mir_descr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
- link robotiq_85_base_link: geometry collision mesh filename=/mnt/data/mir_isaac/install/robotiq_description/share/robot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; visual mesh filename=/mnt/data/mir_isaac/install/robotiq_description/share/robot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
- link robotiq_85_left_finger_link: geometry collision mesh filename=/mnt/data/mir_isaac/install/robotiq_description/share/robot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; visual mesh filename=/mnt/data/mir_isaac/install/robotiq_description/share/robot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
- link robotiq_85_left_finger_tip_link: geometry collision mesh filename=/mnt/data/mir_isaac/install/robotiq_description/share/robot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; visual mesh filename=/mnt/data/mir_isaac/install/robotiq_description/share/robot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
- link robotiq_85_left_inner_knuckle_link: geometry collision mesh filename=/mnt/data/mir_isaac/install/robotiq_description/share/robot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; visual mesh filename=/mnt/data/mir_isaac/install/robotiq_description/share/robot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
- link robotiq_85_left_knuckle_link: geometry collision mesh filename=/mnt/data/mir_isaac/install/robotiq_description/share/robot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; visual mesh filename=/mnt/data/mir_isaac/install/robotiq_description/share/robot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
- link robotiq_85_right_finger_link: geometry collision mesh filename=/mnt/data/mir_isaac/install/robotiq_description/share/robot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; visual mesh filename=/mnt/data/mir_isaac/install/robotiq_description/share/robot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
- link robotiq_85_right_finger_tip_link: geometry collision mesh filename=/mnt/data/mir_isaac/install/robotiq_description/share/robot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; visual mesh filename=/mnt/data/mir_isaac/install/robotiq_description/share/robot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
- link robotiq_85_right_inner_knuckle_link: geometry collision mesh filename=/mnt/data/mir_isaac/install/robotiq_description/share/robot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; visual mesh filename=/mnt/data/mir_isaac/install/robotiq_description/share/robot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
- link robotiq_85_right_knuckle_link: geometry collision mesh filename=/mnt/data/mir_isaac/install/robotiq_description/share/robot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; visual mesh filename=/mnt/data/mir_isaac/install/robotiq_description/share/robot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
- link ur_base_link_inertia: geometry collision mesh filename=/mnt/data/mir_isaac/install/ur_description/share/ur_descrip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; visual mesh filename=/mnt/data/mir_isaac/install/ur_description/share/ur_descrip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
- link ur_forearm_link: geometry collision mesh filename=/mnt/data/mir_isaac/install/ur_description/share/ur_descrip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; visual mesh filename=/mnt/data/mir_isaac/install/ur_description/share/ur_descrip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
- link ur_shoulder_link: geometry collision mesh filename=/mnt/data/mir_isaac/install/ur_description/share/ur_descrip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; visual mesh filename=/mnt/data/mir_isaac/install/ur_description/share/ur_descrip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
- link ur_upper_arm_link: geometry collision mesh filename=/mnt/data/mir_isaac/install/ur_description/share/ur_descrip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; visual mesh filename=/mnt/data/mir_isaac/install/ur_description/share/ur_descrip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
- link ur_wrist_1_link: geometry collision mesh filename=/mnt/data/mir_isaac/install/ur_description/share/ur_descrip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; visual mesh filename=/mnt/data/mir_isaac/install/ur_description/share/ur_descrip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
- link ur_wrist_2_link: geometry collision mesh filename=/mnt/data/mir_isaac/install/ur_description/share/ur_descrip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; visual mesh filename=/mnt/data/mir_isaac/install/ur_description/share/ur_descrip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
- link ur_wrist_3_link: geometry collision mesh filename=/mnt/data/mir_isaac/install/ur_description/share/ur_descrip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; visual mesh filename=/mnt/data/mir_isaac/install/ur_description/share/ur_descrip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
Joints:
- joint left_wheel_joint: limit effort=100 velocity=20.0 -> effort=100 velocity=24.0
- joint right_wheel_joint: limit effort=100 velocity=20.0 -> effort=100 velocity=24.0

File: isaac_sim/mir_isaac_raw.urdf (robot description, URDF)
Before this commit: robot mir_100, 58 links, 57 joints
Links:
- link realsense_link: geometry collision box size=0.02505 0.09 0.025; visual mesh filename=file:///mnt/data/mir_isaac/install/realsense2_description/s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
Joints:
- joint left_wheel_joint: limit effort=100 velocity=20.0 -> effort=100 velocity=24.0
- joint right_wheel_joint: limit effort=100 velocity=20.0 -> effort=100 velocity=24.0

Commit message: feat: add Robotiq FT300 and wrist camera to mobile manipulator
Mount the FT300, wrist camera and 2F-85 in order, including the 55 mm gripper offset. Replace the interfering D435i assembly and update MoveIt collision settings.

Apply black URDF materials to Isaac USD, add an assembly measurement tool, and refresh model previews and documentation.

Validated ROS package builds, URDF parsing, collision checks, gripper-frame FK/IK, OMPL planning and simulated trajectory execution, plus a 120-frame Isaac smoke test.

File: isaac_sim/mir_isaac.urdf (robot description, URDF)
Before this commit: robot mir_100, 58 links, 57 joints
Links:
- removed link camera_mount
- removed link realsense_accel_frame
- removed link realsense_accel_optical_frame
- removed link realsense_bottom_screw_frame
- removed link realsense_color_frame
- removed link realsense_color_optical_frame
- removed link realsense_depth_frame
- removed link realsense_depth_optical_frame
- removed link realsense_gyro_frame
- removed link realsense_gyro_optical_frame
- removed link realsense_infra1_frame
- removed link realsense_infra1_optical_frame
- removed link realsense_infra2_frame
- removed link realsense_infra2_optical_frame
- removed link realsense_link
- added link robotiq_ft300_mounting_plate, mass 0.030; collision cylinder length=0.013 radius=0.0375; visual mesh filename=/mnt/data/mir_isaac/install/mir_description/share/mir_descr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
- added link robotiq_ft300_sensor, mass 0.300; collision cylinder length=0.0348 radius=0.0375; visual mesh filename=/mnt/data/mir_isaac/install/mir_description/share/mir_descr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
- added link robotiq_ft_frame
- added link robotiq_wrist_camera_link, mass 0.160; collision box size=0.045 0.020 0.0224; collision cylinder length=0.0135 radius=0.0375
- added link robotiq_wrist_camera_optical_frame
- added link robotiq_wrist_camera_tool_link
Joints:
- removed joint camera_mount_joint
- removed joint realsense_accel_joint
- removed joint realsense_accel_optical_joint
- removed joint realsense_color_joint
- removed joint realsense_color_optical_joint
- removed joint realsense_depth_joint
- removed joint realsense_depth_optical_joint
- removed joint realsense_gyro_joint
- removed joint realsense_gyro_optical_joint
- removed joint realsense_infra1_joint
- removed joint realsense_infra1_optical_joint
- removed joint realsense_infra2_joint
- removed joint realsense_infra2_optical_joint
- removed joint realsense_joint
- removed joint realsense_link_joint
- added joint robotiq_ft300_mount_joint: type fixed, parent ur_tool0, child robotiq_ft300_mounting_plate
- added joint robotiq_ft300_sensor_joint: type fixed, parent robotiq_ft300_mounting_plate, child robotiq_ft300_sensor, origin xyz=0 0 0.0415
- added joint robotiq_ft_frame_joint: type fixed, parent robotiq_ft300_sensor, child robotiq_ft_frame, origin rpy=0 0 1.5707963267948966
- added joint robotiq_wrist_camera_joint: type fixed, parent robotiq_ft300_sensor, child robotiq_wrist_camera_link
- added joint robotiq_wrist_camera_optical_joint: type fixed, parent robotiq_wrist_camera_link, child robotiq_wrist_camera_optical_frame, origin xyz=0 0.0357 0.0001 rpy=0.5235987755982988 0 0
- added joint robotiq_wrist_camera_tool_joint: type fixed, parent robotiq_wrist_camera_link, child robotiq_wrist_camera_tool_link, origin xyz=0 0 0.0135
- joint robotiq_85_base_joint: parent ur_tool0 -> robotiq_wrist_camera_tool_link

File: isaac_sim/mir_isaac_raw.urdf (robot description, URDF)
Before this commit: robot mir_100, 58 links, 57 joints
Links:
- removed link camera_mount
- removed link realsense_accel_frame
- removed link realsense_accel_optical_frame
- removed link realsense_bottom_screw_frame
- removed link realsense_color_frame
- removed link realsense_color_optical_frame
- removed link realsense_depth_frame
- removed link realsense_depth_optical_frame
- removed link realsense_gyro_frame
- removed link realsense_gyro_optical_frame
- removed link realsense_infra1_frame
- removed link realsense_infra1_optical_frame
- removed link realsense_infra2_frame
- removed link realsense_infra2_optical_frame
- removed link realsense_link
- added link robotiq_ft300_mounting_plate, mass 0.030; collision cylinder length=0.013 radius=0.0375; visual mesh filename=package://mir_description/meshes/robotiq_wrist/robotiq_ft30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
- added link robotiq_ft300_sensor, mass 0.300; collision cylinder length=0.0348 radius=0.0375; visual mesh filename=package://mir_description/meshes/robotiq_wrist/robotiq_ft30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
- added link robotiq_ft_frame
- added link robotiq_wrist_camera_link, mass 0.160; collision box size=0.045 0.020 0.0224; collision cylinder length=0.0135 radius=0.0375
- added link robotiq_wrist_camera_optical_frame
- added link robotiq_wrist_camera_tool_link
Joints:
- removed joint camera_mount_joint
- removed joint realsense_accel_joint
- removed joint realsense_accel_optical_joint
- removed joint realsense_color_joint
- removed joint realsense_color_optical_joint
- removed joint realsense_depth_joint
- removed joint realsense_depth_optical_joint
- removed joint realsense_gyro_joint
- removed joint realsense_gyro_optical_joint
- removed joint realsense_infra1_joint
- removed joint realsense_infra1_optical_joint
- removed joint realsense_infra2_joint
- removed joint realsense_infra2_optical_joint
- removed joint realsense_joint
- removed joint realsense_link_joint
- added joint robotiq_ft300_mount_joint: type fixed, parent ur_tool0, child robotiq_ft300_mounting_plate
- added joint robotiq_ft300_sensor_joint: type fixed, parent robotiq_ft300_mounting_plate, child robotiq_ft300_sensor, origin xyz=0 0 0.0415
- added joint robotiq_ft_frame_joint: type fixed, parent robotiq_ft300_sensor, child robotiq_ft_frame, origin rpy=0 0 1.5707963267948966
- added joint robotiq_wrist_camera_joint: type fixed, parent robotiq_ft300_sensor, child robotiq_wrist_camera_link
- added joint robotiq_wrist_camera_optical_joint: type fixed, parent robotiq_wrist_camera_link, child robotiq_wrist_camera_optical_frame, origin xyz=0 0.0357 0.0001 rpy=0.5235987755982988 0 0
- added joint robotiq_wrist_camera_tool_joint: type fixed, parent robotiq_wrist_camera_link, child robotiq_wrist_camera_tool_link, origin xyz=0 0 0.0135
- joint robotiq_85_base_joint: parent ur_tool0 -> robotiq_wrist_camera_tool_link

File: mir_robot/mir_description/urdf/include/mir_100_v1.urdf.xacro (robot description, xacro)
@@ -6,5 +6,4 @@
   <xacro:include filename="$(find mir_description)/urdf/include/wheel.urdf.xacro" />
   <xacro:include filename="$(find mir_description)/urdf/include/caster.urdf.xacro" />
-  <xacro:include filename="$(find realsense2_description)/urdf/_d435i.urdf.xacro"/>
   <xacro:property name="deg_to_rad" value="0.017453293" />
   <!-- The inertia for the MiR platform is intentionally chosen to be smaller than
@@ -317,38 +316,13 @@
       </gazebo>
     </xacro:if>
-    <link name="${prefix}camera_mount">
-      <visual>
-        <origin xyz="0 0 0" rpy="0 0 0" />
-        <geometry>
-          <mesh filename="package://mir_description/meshes/visual/D435i_mounted.STL" scale="0.001 0.001 0.001" />
-        </geometry>
-        <xacro:insert_block name="material_light_grey" />
-      </visual>
-      <collision>
-        <origin xyz="0 0 0" rpy="0 0 0" />
-        <geometry>
-          <mesh filename="package://mir_description/meshes/collision/D435i_mounted.STL" scale="0.001 0.001 0.001" />
-        </geometry>
-      </collision>
-    </link>
-    <joint name="${prefix}camera_mount_joint" type="fixed">
-      <parent link="ur_flange" />
-      <child link="${prefix}camera_mount" />
-      <origin xyz="0.035 0.05 0.03" rpy="0 ${pi} ${0.5 * pi}" />
-    </joint>
-    <!-- realsense_gazebo_plugin is off by default: it throws during Load and
-         regularly segfaults gzserver right afterwards, while never actually
-         publishing colour or depth. Pass realsense_gazebo_plugin:=true if you
-         have a working build of it. -->
-    <xacro:arg name="realsense_gazebo_plugin" default="false" />
-    <xacro:sensor_d435i parent="ur_flange" name="realsense" use_nominal_extrinsics="true"
-                        add_gazebo_plugin="$(arg realsense_gazebo_plugin)">
-      <origin xyz="0.02 0 -0.061" rpy="${pi} 0 0"/>
-    </xacro:sensor_d435i>
+    <!-- The former flange-mounted D435i bracket intersects the FT300.
+         The Robotiq Wrist Camera below replaces that wrist camera assembly. -->
     <xacro:arg name="use_fake_hardware" default="true" />
   <xacro:arg name="com_port" default="/dev/ttyUSB0" />
   <!-- Import gripper macros -->
+  <xacro:include filename="$(find mir_description)/urdf/include/robotiq_wrist_stack.xacro" />
+  <xacro:robotiq_wrist_stack parent="ur_tool0" />
   <xacro:include filename="$(find mir_description)/urdf/include/robotiq_gripper_macro.xacro" />
-  <xacro:robotiq_gripper name="RobotiqGripperHardwareInterface" prefix="" parent="ur_tool0" use_fake_hardware="$(arg use_fake_hardware)" com_port="$(arg com_port)" sim_gazebo="$(arg sim_gazebo)" sim_isaac="$(arg sim_isaac)" isaac_joint_commands="/isaac_gripper_commands" isaac_joint_states="$(arg isaac_joint_states)">
+  <xacro:robotiq_gripper name="RobotiqGripperHardwareInterface" prefix="" parent="robotiq_wrist_camera_tool_link" use_fake_hardware="$(arg use_fake_hardware)" com_port="$(arg com_port)" sim_gazebo="$(arg sim_gazebo)" sim_isaac="$(arg sim_isaac)" isaac_joint_commands="/isaac_gripper_commands" isaac_joint_states="$(arg isaac_joint_states)">
     <origin xyz="0 0 0" rpy="0 0 0" />
   </xacro:robotiq_gripper>
