Commit message: fix: restore D435i alongside the Robotiq wrist camera
Relocate the original D435i and bracket to the gripper-side mounting face, preserving their gripper-relative transforms and the 55 mm wrist stack offset.

Restore the camera and bracket in MoveIt with mating-surface collision exclusions. Regenerate the dual-camera URDF/USD, previews and documentation.

Validated both URDF variants, 51 collision configurations, camera transforms, and MoveIt FK/IK, planning and simulated trajectory execution.

File: isaac_sim/mir_isaac.urdf (robot description, URDF)
Before this commit: robot mir_100, 49 links, 48 joints
Links:
- added link camera_mount; collision mesh filename=/mnt/data/mir_isaac/install/mir_description/share/mir_descr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 scale=0.001 0.001 0.001; visual mesh filename=/mnt/data/mir_isaac/install/mir_description/share/mir_descr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 scale=0.001 0.001 0.001
- added link d435i_mount_frame
- added link realsense_accel_frame
- added link realsense_accel_optical_frame
- added link realsense_bottom_screw_frame
- added link realsense_color_frame
- added link realsense_color_optical_frame
- added link realsense_depth_frame
- added link realsense_depth_optical_frame
- added link realsense_gyro_frame
- added link realsense_gyro_optical_frame
- added link realsense_infra1_frame
- added link realsense_infra1_optical_frame
- added link realsense_infra2_frame
- added link realsense_infra2_optical_frame
- added link realsense_link, mass 0.072; collision box size=0.02505 0.09 0.025; visual mesh filename=/mnt/data/mir_isaac/install/realsense2_description/share/re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
Joints:
- added joint camera_mount_joint: type fixed, parent d435i_mount_frame, child camera_mount, origin xyz=0.035 0.05 0.03 rpy=0 3.141592653589793 1.5707963267948966
- added joint d435i_mount_frame_joint: type fixed, parent robotiq_wrist_camera_tool_link, child d435i_mount_frame, origin xyz=0 0 0 rpy=-1.5707963267948966 -1.5707963267948966 0
- added joint realsense_accel_joint: type fixed, parent realsense_link, child realsense_accel_frame, origin xyz=-0.01174 -0.00552 0.0051 rpy=0 0 0
- added joint realsense_accel_optical_joint: type fixed, parent realsense_accel_frame, child realsense_accel_optical_frame, origin xyz=0 0 0 rpy=-1.5707963267948966 0 -1.5707963267948966
- added joint realsense_color_joint: type fixed, parent realsense_link, child realsense_color_frame, origin xyz=0 0.015 0 rpy=0 0 0
- added joint realsense_color_optical_joint: type fixed, parent realsense_color_frame, child realsense_color_optical_frame, origin xyz=0 0 0 rpy=-1.5707963267948966 0 -1.5707963267948966
- added joint realsense_depth_joint: type fixed, parent realsense_link, child realsense_depth_frame, origin xyz=0 0 0 rpy=0 0 0
- added joint realsense_depth_optical_joint: type fixed, parent realsense_depth_frame, child realsense_depth_optical_frame, origin xyz=0 0 0 rpy=-1.5707963267948966 0 -1.5707963267948966
- added joint realsense_gyro_joint: type fixed, parent realsense_link, child realsense_gyro_frame, origin xyz=-0.01174 -0.00552 0.0051 rpy=0 0 0
- added joint realsense_gyro_optical_joint: type fixed, parent realsense_gyro_frame, child realsense_gyro_optical_frame, origin xyz=0 0 0 rpy=-1.5707963267948966 0 -1.5707963267948966
- added joint realsense_infra1_joint: type fixed, parent realsense_link, child realsense_infra1_frame, origin xyz=0 0.0 0 rpy=0 0 0
- added joint realsense_infra1_optical_joint: type fixed, parent realsense_infra1_frame, child realsense_infra1_optical_frame, origin xyz=0 0 0 rpy=-1.5707963267948966 0 -1.5707963267948966
- added joint realsense_infra2_joint: type fixed, parent realsense_link, child realsense_infra2_frame, origin xyz=0 -0.05 0 rpy=0 0 0
- added joint realsense_infra2_optical_joint: type fixed, parent realsense_infra2_frame, child realsense_infra2_optical_frame, origin xyz=0 0 0 rpy=-1.5707963267948966 0 -1.5707963267948966
- added joint realsense_joint: type fixed, parent d435i_mount_frame, child realsense_bottom_screw_frame, origin xyz=0.02 0 -0.061 rpy=3.141592653589793 0 0
- added joint realsense_link_joint: type fixed, parent realsense_bottom_screw_frame, child realsense_link, origin xyz=0.010600000000000002 0.0175 0.0125 rpy=0 0 0

File: isaac_sim/mir_isaac_raw.urdf (robot description, URDF)
Before this commit: robot mir_100, 49 links, 48 joints
Links:
- added link camera_mount; collision mesh filename=package://mir_description/meshes/collision/D435i_mounted.STL scale=0.001 0.001 0.001; visual mesh filename=package://mir_description/meshes/visual/D435i_mounted.STL scale=0.001 0.001 0.001
- added link d435i_mount_frame
- added link realsense_accel_frame
- added link realsense_accel_optical_frame
- added link realsense_bottom_screw_frame
- added link realsense_color_frame
- added link realsense_color_optical_frame
- added link realsense_depth_frame
- added link realsense_depth_optical_frame
- added link realsense_gyro_frame
- added link realsense_gyro_optical_frame
- added link realsense_infra1_frame
- added link realsense_infra1_optical_frame
- added link realsense_infra2_frame
- added link realsense_infra2_optical_frame
- added link realsense_link, mass 0.072; collision box size=0.02505 0.09 0.025; visual mesh filename=file:///mnt/data/mir_isaac/install/realsense2_description/s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
Joints:
- added joint camera_mount_joint: type fixed, parent d435i_mount_frame, child camera_mount, origin xyz=0.035 0.05 0.03 rpy=0 3.141592653589793 1.5707963267948966
- added joint d435i_mount_frame_joint: type fixed, parent robotiq_wrist_camera_tool_link, child d435i_mount_frame, origin xyz=0 0 0 rpy=-1.5707963267948966 -1.5707963267948966 0
- added joint realsense_accel_joint: type fixed, parent realsense_link, child realsense_accel_frame, origin xyz=-0.01174 -0.00552 0.0051 rpy=0 0 0
- added joint realsense_accel_optical_joint: type fixed, parent realsense_accel_frame, child realsense_accel_optical_frame, origin xyz=0 0 0 rpy=-1.5707963267948966 0 -1.5707963267948966
- added joint realsense_color_joint: type fixed, parent realsense_link, child realsense_color_frame, origin xyz=0 0.015 0 rpy=0 0 0
- added joint realsense_color_optical_joint: type fixed, parent realsense_color_frame, child realsense_color_optical_frame, origin xyz=0 0 0 rpy=-1.5707963267948966 0 -1.5707963267948966
- added joint realsense_depth_joint: type fixed, parent realsense_link, child realsense_depth_frame, origin xyz=0 0 0 rpy=0 0 0
- added joint realsense_depth_optical_joint: type fixed, parent realsense_depth_frame, child realsense_depth_optical_frame, origin xyz=0 0 0 rpy=-1.5707963267948966 0 -1.5707963267948966
- added joint realsense_gyro_joint: type fixed, parent realsense_link, child realsense_gyro_frame, origin xyz=-0.01174 -0.00552 0.0051 rpy=0 0 0
- added joint realsense_gyro_optical_joint: type fixed, parent realsense_gyro_frame, child realsense_gyro_optical_frame, origin xyz=0 0 0 rpy=-1.5707963267948966 0 -1.5707963267948966
- added joint realsense_infra1_joint: type fixed, parent realsense_link, child realsense_infra1_frame, origin xyz=0 0.0 0 rpy=0 0 0
- added joint realsense_infra1_optical_joint: type fixed, parent realsense_infra1_frame, child realsense_infra1_optical_frame, origin xyz=0 0 0 rpy=-1.5707963267948966 0 -1.5707963267948966
- added joint realsense_infra2_joint: type fixed, parent realsense_link, child realsense_infra2_frame, origin xyz=0 -0.05 0 rpy=0 0 0
- added joint realsense_infra2_optical_joint: type fixed, parent realsense_infra2_frame, child realsense_infra2_optical_frame, origin xyz=0 0 0 rpy=-1.5707963267948966 0 -1.5707963267948966
- added joint realsense_joint: type fixed, parent d435i_mount_frame, child realsense_bottom_screw_frame, origin xyz=0.02 0 -0.061 rpy=3.141592653589793 0 0
- added joint realsense_link_joint: type fixed, parent realsense_bottom_screw_frame, child realsense_link, origin xyz=0.010600000000000002 0.0175 0.0125 rpy=0 0 0

File: mir_robot/mir_description/urdf/include/mir_100_v1.urdf.xacro (robot description, xacro)
@@ -6,4 +6,5 @@
   <xacro:include filename="$(find mir_description)/urdf/include/wheel.urdf.xacro" />
   <xacro:include filename="$(find mir_description)/urdf/include/caster.urdf.xacro" />
+  <xacro:include filename="$(find realsense2_description)/urdf/_d435i.urdf.xacro"/>
   <xacro:property name="deg_to_rad" value="0.017453293" />
   <!-- The inertia for the MiR platform is intentionally chosen to be smaller than
@@ -316,6 +317,43 @@
       </gazebo>
     </xacro:if>
-    <!-- The former flange-mounted D435i bracket intersects the FT300.
-         The Robotiq Wrist Camera below replaces that wrist camera assembly. -->
+    <!-- Preserve the original D435i/bracket geometry relative to the gripper.
+         Mount on the tool side of the wrist stack, 55 mm beyond the original
+         flange position. This frame undoes flange->tool0 rotation, allowing
+         the original camera/bracket mounting coordinates to stay unchanged. -->
+    <link name="${prefix}d435i_mount_frame" />
+    <joint name="${prefix}d435i_mount_frame_joint" type="fixed">
+      <parent link="robotiq_wrist_camera_tool_link" />
+      <child link="${prefix}d435i_mount_frame" />
+      <origin xyz="0 0 0" rpy="${-pi/2} ${-pi/2} 0" />
+    </joint>
+    <link name="${prefix}camera_mount">
+      <visual>
+        <origin xyz="0 0 0" rpy="0 0 0" />
+        <geometry>
+          <mesh filename="package://mir_description/meshes/visual/D435i_mounted.STL" scale="0.001 0.001 0.001" />
+        </geometry>
+        <xacro:insert_block name="material_light_grey" />
+      </visual>
+      <collision>
+        <origin xyz="0 0 0" rpy="0 0 0" />
+        <geometry>
+          <mesh filename="package://mir_description/meshes/collision/D435i_mounted.STL" scale="0.001 0.001 0.001" />
+        </geometry>
+      </collision>
+    </link>
+    <joint name="${prefix}camera_mount_joint" type="fixed">
+      <parent link="${prefix}d435i_mount_frame" />
+      <child link="${prefix}camera_mount" />
+      <origin xyz="0.035 0.05 0.03" rpy="0 ${pi} ${0.5 * pi}" />
+    </joint>
+    <!-- realsense_gazebo_plugin is off by default: it throws during Load and
+         regularly segfaults gzserver right afterwards, while never actually
+         publishing colour or depth. Pass realsense_gazebo_plugin:=true if you
+         have a working build of it. -->
+    <xacro:arg name="realsense_gazebo_plugin" default="false" />
+    <xacro:sensor_d435i parent="${prefix}d435i_mount_frame" name="realsense" use_nominal_extrinsics="true"
+                        add_gazebo_plugin="$(arg realsense_gazebo_plugin)">
+      <origin xyz="0.02 0 -0.061" rpy="${pi} 0 0"/>
+    </xacro:sensor_d435i>
     <xacro:arg name="use_fake_hardware" default="true" />
   <xacro:arg name="com_port" default="/dev/ttyUSB0" />
